File: pcb/ftdi.sch (KiCad schematic (older format))
At the start: 44 parts

Commit message: primer versión terminada del esquemático
Parts:
- gave numbers to parts that had none: 42
Other:
- moved on the sheet: C10, C18, C9, FB1, FB2

Commit message: - se agregan todos los footprints
Parts:
- C10, C11, C12, C13, C14, C15, C16, C17, C18, C19, C20, C21, C5, C6, C9: footprint (none) -> Capacitor_SMD:C_0603_1608Metric
- D3, D4: footprint (none) -> LED_SMD:LED_0603_1608Metric
- D5, D6: footprint (none) -> Diode_SMD:D_0603_1608Metric
- FB1, FB2: footprint (none) -> Inductor_SMD:L_0603_1608Metric
- IC1: footprint SOIC127P600X175-8N -> SamacSys_Parts:SOIC127P600X175-8N
- IC2: footprint SOT65P210X110-5N -> SamacSys_Parts:SOT65P210X110-5N
- IC3: footprint QFN50P250X300X100-15N-D -> SamacSys_Parts:QFN50P250X300X100-15N-D
- R10, R11, R12, R13, R14, R15, R16, R17, R18, R19, R20, R21, R22, R6, R7, R8, R9: footprint (none) -> Resistor_SMD:R_0603_1608Metric
- Y1: footprint ECS3201233AGMTR -> Crystal:Crystal_SMD_0603-4Pin_6.0x3.5mm

Commit message: - Se agregan hojas de datos e información del proyecto.
Parts:
- renumbered IC1 to U3, IC2 to U4, IC3 to U5
Changed lines of the file:
@@
 encoding utf-8
 Sheet 2 2
-Title ""
+Title "Espressif Programmer"
 Date ""
-Rev ""
-Comp ""
-Comment1 ""
-Comment2 ""
+Rev "1.1"
+Comp "Sipel SRL"
+Comment1 "Autor: Gonzalo Sanhez"
+Comment2 "Licencia: Open source hardware"
 Comment3 ""
 Comment4 ""
@@
 	3250 1950 2600 1950
 $Comp
-L SamacSys_Parts:M93C46-WMN6TP IC1
+L SamacSys_Parts:M93C46-WMN6TP U3
 U 1 1 60E7BE25
 P 2400 6850
-F 0 "IC1" H 2850 7115 50  0000 C CNN
+F 0 "U3" H 2850 7115 50  0000 C CNN
 F 1 "M93C46-WMN6TP" H 2850 7024 50  0000 C CNN
 F 2 "SamacSys_Parts:SOIC127P600X175-8N" H 3150 6950 50  0001 L CNN
@@
 EEDATA
 $Comp
-L SamacSys_Parts:74AHC125BQ,115 IC3
+L SamacSys_Parts:74AHC125BQ,115 U5
 U 1 1 60ED1A1F
 P 8950 4850
-F 0 "IC3" H 9750 3950 50  0000 C CNN
+F 0 "U5" H 9750 3950 50  0000 C CNN
 F 1 "74AHC125BQ,115" H 10000 4050 50  0000 C CNN
 F 2 "SamacSys_Parts:QFN50P250X300X100-15N-D" H 10000 5250 50  0001 L CNN
@@
 FT_TCK
 $Comp
-L SamacSys_Parts:MC74VHC1GT04DFT1 IC2
+L SamacSys_Parts:MC74VHC1GT04DFT1 U4
 U 1 1 60F0B678
 P 8850 3100
-F 0 "IC2" H 9450 3365 50  0000 C CNN
+F 0 "U4" H 9450 3365 50  0000 C CNN
 F 1 "MC74VHC1GT04DFT1" H 9450 3274 50  0000 C CNN
 F 2 "SamacSys_Parts:SOT65P210X110-5N" H 9900 3200 50  0001 L CNN
